File: Eagle Files/SensochSens/Cleanup/Sen_final.brd (EAGLE design)
At the start: 63.5 x 50.5 mm, 36 parts, among them U1 SM700PC1SMD, U2 MIC5219, U3 KCSA03-102SMD_7SEG

Commit message: cleanup
Parts:
- removed S3: Primary sw, switch:A68-A31
- added PRIMARY_SW: S3, cy-con:SS-22
- C1: device SparkFun-Passives:0603-CAP -> SparkFun-Passives:0805
- C4: device SparkFun-Passives:0402-CAP -> SparkFun-Passives:0805
- moved JP8 20.3 mm to (24.1, 3.81)
- moved R7 8.13 mm to (2.54, 41.9)
- moved JP4 6.35 mm to (10.2, 3.81)
- moved U3 2.54 mm to (15.2, 45.7)
- moved R6 1.27 mm to (25.4, 47.0)
- moved DIV_ID 1.27 mm to (57.1, 14.0)
- moved JP10 1.27 mm to (39.4, 47.0)
- turned LED1 to 180 degrees
- turned LED2 to 180 degrees
- turned LED3 to 180 degrees
- turned LED4 to 180 degrees
Connections:
- net ADC1: now also JP4.4; no longer JP4.3
- net ADC2: now also JP4.6; no longer JP4.4
- net ADC3: now also JP4.8; no longer JP4.5
- net ADC4: now also JP4.3; no longer JP4.6
- net ADC5: now also JP4.5; no longer JP4.7
- net ADC6: now also JP4.7; no longer JP4.8
- net EN: now also PRIMARY_SW.5; no longer S3.5
- net GND: now also PRIMARY_SW.6; no longer S3.6
- net VBATT: now also PRIMARY_SW.2, PRIMARY_SW.4; no longer S3.2, S3.4
- net VCC1: now also PRIMARY_SW.1; no longer S3.1
Routing:
- net GND: track 214.9 -> 258.3 mm, vias 1 -> 0
- net 3.3V: track 258.7 -> 237.3 mm, vias 5 -> 0
- net CH_4: track 42.4 -> 23.0 mm, vias 1 -> 0
- net ADC4: track 8.74 -> 24.7 mm
- net VCC1: track 19.0 -> 33.2 mm, vias 1 -> 0
- net TOGL: track 33.8 -> 44.9 mm
- net DIV_1: track 51.1 -> 62.0 mm, vias 1 -> 0
- net ADC1: track 22.1 -> 11.4 mm
- net EN: track 27.6 -> 16.9 mm
- net ADC3: track 17.7 -> 8.82 mm, vias 1 -> 0
- net ADC0: track 21.4 -> 12.6 mm, vias 1 -> 0
- net DIV_2: track 41.3 -> 49.8 mm
- net CH_2: track 29.0 -> 21.2 mm
- net SCL: track 35.2 -> 27.5 mm, vias 2 -> 1
- net ADC6: track 8.53 -> 15.6 mm
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- added copper zone on layer 1, net GND
- added copper zone on layer 16, net GND
