File: Eagle Files/SensochSens/Cleanup/Sen_final.sch (EAGLE design)
At the start: 29 parts, among them U1 SM700PC1SMD, U2 MIC5219, X2 ADC0-7

Commit message: cleanup
Parts:
- removed S3: (no value), switch:A68-A31
- removed X2: ADC0-7, con-molex:53047-10
- added JP4: M05X2SHD_LOCK, SparkFun-Connectors:M05X2SHD_LOCK
- added PRIMARY_SW: S3, cy-con:SS22_SD
- C1, C4: device SparkFun-Passives:CAP0402-CAP -> SparkFun-Passives:CAP0805
- C2, C3: device SparkFun-Passives:CAP_POL1206 -> SparkFun-Passives:CAP_POL3528
- CH, DIV_ID: value (none) -> HIX DIP
- JP2: value LIPO_charger -> LIPO
- R1, R2: device SparkFun-Passives:RESISTOR0402-RES -> SparkFun-Passives:RESISTOR0805-RES
- R3, R4, R5, R6, R7: device SparkFun-Passives:RESISTOR0402-RES -> SparkFun-Passives:RESISTOR0603-RES
- S1: value (none) -> Secondary sw
- renumbered U$1 to U3
Connections:
- net 3.3V: now also JP4.1, JP4.10; no longer X2-1.S, X2-2.S
- net ADC0: now also JP4.2; no longer X2-3.S
- net ADC1: now also JP4.4; no longer X2-4.S
- net ADC2: now also JP4.6; no longer X2-5.S
- net ADC3: now also JP4.8; no longer X2-6.S
- net ADC4: now also JP4.3; no longer X2-7.S
- net ADC5: now also JP4.5; no longer X2-8.S
- net ADC6: now also JP4.7; no longer X2-9.S
- net ADC7: now also JP4.9; no longer X2-10.S
- net EN: now also PRIMARY_SW.5; no longer S3B.P
- net GND: now also PRIMARY_SW.6; no longer S3B.S
- net VBATT: now also PRIMARY_SW.2, PRIMARY_SW.4; no longer S3A.P, S3B.O
- net VCC1: now also PRIMARY_SW.1; no longer S3A.O
Other:
- note added: "Design by: Kartik Karuna (Kartik@kth.se)"
- note removed: "Design by : Kartik Karuna (Kartik@kth.se)"
